Commit message: xacro

File: amr_dd/models/amr_dd.xacro (robot description, xacro)
@@ -1,68 +1,7 @@
 <?xml version='1.0'?>
-<robot name="m2wr" xmlns:xacro="http://www.ros.org/wiki/xacro">
-    <material name="black">
-        <color rgba="0.0 0.0 0.0 1.0"/>
-    </material>
-    <material name="blue">
-        <color rgba="0.203125 0.23828125 0.28515625 1.0"/>
-    </material>
-    <material name="green">
-        <color rgba="0.0 0.8 0.0 1.0"/>
-    </material>
-    <material name="grey">
-        <color rgba="0.2 0.2 0.2 1.0"/>
-    </material>
-    <material name="orange">
-        <color rgba="1.0 0.423529411765 0.0392156862745 1.0"/>
-    </material>
-    <material name="brown">
-        <color rgba="0.870588235294 0.811764705882 0.764705882353 1.0"/>
-    </material>
-    <material name="red">
-        <color rgba="0.80078125 0.12890625 0.1328125 1.0"/>
-    </material>
-    <material name="white">
-        <color rgba="1.0 1.0 1.0 1.0"/>
-    </material>
-    <gazebo reference="chassis">
-        <material>Gazebo/Orange</material>
-    </gazebo>
-    <gazebo reference="left_wheel">
-        <material>Gazebo/Blue</material>
-    </gazebo>
-    <gazebo reference="right_wheel">
-        <material>Gazebo/Blue</material>
-    </gazebo>
-    <gazebo reference="hook">
-        <material>Gazebo/Green</material>
-    </gazebo>
-    <gazebo reference="cart">
-        <material>Gazebo/Black</material>
-    </gazebo>
-    <gazebo reference="left_cart_wheel">
-        <material>Gazebo/Red</material>
-    </gazebo>
-    <gazebo reference="right_cart_wheel">
-        <material>Gazebo/Red</material>
-    </gazebo>
-    <gazebo>
-        <plugin filename="libgazebo_ros_diff_drive.so" name="differential_drive_controller">
-            <legacyMode>false</legacyMode>
-            <alwaysOn>true</alwaysOn>
-            <updateRate>20</updateRate>
-            <leftJoint>joint_left_wheel</leftJoint>
-            <rightJoint>joint_right_wheel</rightJoint>
-            <wheelSeparation>0.76</wheelSeparation>
-            <wheelDiameter>0.16</wheelDiameter>
-            <torque>0.1</torque>
-            <commandTopic>cmd_vel</commandTopic>
-            <odometryTopic>odom</odometryTopic>
-            <odometryFrame>odom</odometryFrame>
-            <robotBaseFrame>chassis</robotBaseFrame>
-        </plugin>
-        <plugin name="gazebo_ros_control" filename="libgazebo_ros_control.so">
-            <robotNamespace>/amr_dd</robotNamespace>
-        </plugin>
-    </gazebo>
+<robot name="amr_dd" xmlns:xacro="http://www.ros.org/wiki/xacro">
+    <xacro:include filename="$(find amr_dd)/models/materials.xacro" />
+    <xacro:include filename="$(find amr_dd)/models/amr_dd.gazebo" />
+    <xacro:include filename="$(find amr_dd)/models/macros.xacro" />
     <link name='chassis'>
         <!-- pose and inertial -->
@@ -233,23 +172,5 @@
     </link>
     <!-- AMR Wheel -->
-    <link name="left_wheel">
-        <inertial>
-            <mass value="0.2"/>
-            <origin rpy="0 1.5707 1.5707" xyz="0 0 0"/>
-            <inertia ixx="0.000526666666667" ixy="0" ixz="0" iyy="0.000526666666667" iyz="0" izz="0.001"/>
-        </inertial>
-        <collision name="left_wheel_collision">
-            <origin rpy="0 1.5707 1.5707" xyz="0 0 0"/>
-            <geometry>
-                <cylinder length="0.05" radius="0.08"/>
-            </geometry>
-        </collision>
-        <visual name="left_wheel_visual">
-            <origin rpy="0 1.5707 1.5707" xyz="0 0 0"/>
-            <geometry>
-                <cylinder length="0.05" radius="0.08"/>
-            </geometry>
-        </visual>
-    </link>
+    <xacro:link_wheel name="left_wheel" />
     <gazebo reference="left_wheel">
         <mu1>100000.0</mu1>
@@ -564,19 +485,3 @@
         </actuator>
     </transmission>
-    <!-- <include name="hokuyo">
-        <uri>model://hokuyo</uri>
-        <pose>0.45 0 0.4 0 0 0</pose>
-    </include>
-    <joint type="fixed" name="hokuyo_joint">
-        <child>hokuyo::link</child>
-        <parent>chassis</parent>
-    </joint> -->
-    <!-- <include name="camera">
-        <uri>model://camera</uri>
-        <pose>0.5 0 0.15 0 -0.25 0</pose>
-    </include>
-    <joint type="fixed" name="camera_joint">
-        <child>camera::link</child>
-        <parent>chassis</parent>
-    </joint> -->
 </robot>

Commit message: develop

File: amr_dd/models/amr_dd.xacro (robot description, xacro)
@@ -26,92 +26,8 @@
         </visual>
         <!-- caster -->
-        <collision name='caster_collision_TL'>
-            <origin rpy="0 0 0" xyz="0.45 0.35 -0.135"/>
-            <geometry>
-                <sphere radius="0.05"/>
-            </geometry>
-            <surface>
-                <friction>
-                    <ode>
-                        <mu>0</mu>
-                        <mu2>0</mu2>
-                        <slip1>1.0</slip1>
-                        <slip2>1.0</slip2>
-                    </ode>
-                </friction>
-            </surface>
-            </collision>
-            <visual name='caster_visual_TL'>
-                <origin rpy="0 0 0" xyz="0.45 0.35 -0.135"/>
-                <geometry>
-                    <sphere radius="0.05"/>
-                </geometry>
-            </visual>
-        <collision name='caster_collision_TR'>
-            <origin rpy="0 0 0" xyz="0.45 -0.35 -0.135"/>
-            <geometry>
-                <sphere radius="0.05"/>
-            </geometry>
-            <surface>
-                <friction>
-                    <ode>
-                        <mu>0</mu>
-                        <mu2>0</mu2>
-                        <slip1>1.0</slip1>
-                        <slip2>1.0</slip2>
-                    </ode>
-                </friction>
-            </surface>
-        </collision>
-        <visual name='caster_visual_TR'>
-            <origin rpy="0 0 0" xyz="0.45 -0.35 -0.135"/>
-            <geometry>
-                <sphere radius="0.05"/>
-            </geometry>
-        </visual>
-        <collision name='caster_collision_BL'>
-            <origin rpy="0 0 0" xyz="-0.45 0.35 -0.135"/>
-            <geometry>
-                <sphere radius="0.05"/>
-            </geometry>
-            <surface>
-                <friction>
-                    <ode>
-                        <mu>0</mu>
-                        <mu2>0</mu2>
-                        <slip1>1.0</slip1>
-                        <slip2>1.0</slip2>
-                    </ode>
-                </friction>
-            </surface>
-        </collision>
-        <visual name='caster_visual_BL'>
-            <origin rpy="0 0 0" xyz="-0.45 0.35 -0.135"/>
-            <geometry>
-                <sphere radius="0.05"/>
-            </geometry>
-        </visual>
-        <collision name='caster_collision_BR'>
-            <origin rpy="0 0 0" xyz="-0.45 -0.35 -0.135"/>
-            <geometry>
-                <sphere radius="0.05"/>
-            </geometry>
-            <surface>
-                <friction>
-                    <ode>
-                        <mu>0</mu>
-                        <mu2>0</mu2>
-                        <slip1>1.0</slip1>
-                        <slip2>1.0</slip2>
-                    </ode>
-                </friction>
-            </surface>
-        </collision>
-        <visual name='caster_visual_BR'>
-            <origin rpy="0 0 0" xyz="-0.45 -0.35 -0.135"/>
-            <geometry>
-                <sphere radius="0.05"/>
-            </geometry>
-        </visual>
+        <xacro:caster name="caster_TL" origin_xyz="0.45 0.35 -0.135"/>
+        <xacro:caster name="caster_TR" origin_xyz="0.45 -0.35 -0.135"/>
+        <xacro:caster name="caster_BL" origin_xyz="-0.45 0.35 -0.135"/>
+        <xacro:caster name="caster_BR" origin_xyz="-0.45 -0.35 -0.135"/>
         <collision name='poll_collision'>
             <origin rpy="0 0 0" xyz="0 0 0.25"/>
@@ -181,23 +97,5 @@
         <maxVel>1.0</maxVel>
     </gazebo>
-    <link name="right_wheel">
-        <inertial>
-            <mass value="0.2"/>
-            <origin rpy="0 1.5707 1.5707" xyz="0 0 0"/>
-            <inertia ixx="0.000526666666667" ixy="0" ixz="0" iyy="0.000526666666667" iyz="0" izz="0.001"/>
-        </inertial>
-        <collision name="right_wheel_collision">
-            <origin rpy="0 1.5707 1.5707" xyz="0 0 0"/>
-            <geometry>
-                <cylinder length="0.05" radius="0.08"/>
-            </geometry>
-        </collision>
-        <visual name="right_wheel_visual">
-            <origin rpy="0 1.5707 1.5707" xyz="0 0 0"/>
-            <geometry>
-                <cylinder length="0.05" radius="0.08"/>
-            </geometry>
-        </visual>
-    </link>
+    <xacro:link_wheel name="right_wheel" />
     <gazebo reference="right_wheel">
         <mu1>100000.0</mu1>
@@ -277,113 +175,11 @@
         </visual>
         <!-- caster -->
-        <collision name='cart_caster_collision_TL'>
-            <origin rpy="0 0 0" xyz="-0.95 0.35 -0.135"/>
-            <geometry>
-                <sphere radius="0.05"/>
-            </geometry>
-            <surface>
-                <friction>
-                    <ode>
-                        <mu>0</mu>
-                        <mu2>0</mu2>
-                        <slip1>1.0</slip1>
-                        <slip2>1.0</slip2>
-                    </ode>
-                </friction>
-            </surface>
-            </collision>
-            <visual name='cart_caster_visual_TL'>
-                <origin rpy="0 0 0" xyz="-0.95 0.35 -0.135"/>
-                <geometry>
-                    <sphere radius="0.05"/>
-                </geometry>
-            </visual>
-        <collision name='cart_caster_collision_TR'>
-            <origin rpy="0 0 0" xyz="-0.95 -0.35 -0.135"/>
-            <geometry>
-                <sphere radius="0.05"/>
-            </geometry>
-            <surface>
-                <friction>
-                    <ode>
-                        <mu>0</mu>
-                        <mu2>0</mu2>
-                        <slip1>1.0</slip1>
-                        <slip2>1.0</slip2>
-                    </ode>
-                </friction>
-            </surface>
-        </collision>
-        <visual name='cart_caster_visual_TR'>
-            <origin rpy="0 0 0" xyz="-0.95 -0.35 -0.135"/>
-            <geometry>
-                <sphere radius="0.05"/>
-            </geometry>
-        </visual>
-        <collision name='cart_caster_collision_BL'>
-            <origin rpy="0 0 0" xyz="-1.85 0.35 -0.135"/>
-            <geometry>
-                <sphere radius="0.05"/>
-            </geometry>
-            <surface>
-                <friction>
-                    <ode>
-                        <mu>0</mu>
-                        <mu2>0</mu2>
-                        <slip1>1.0</slip1>
-                        <slip2>1.0</slip2>
-                    </ode>
-                </friction>
-            </surface>
-        </collision>
-        <visual name='cart_caster_visual_BL'>
-            <origin rpy="0 0 0" xyz="-1.85 0.35 -0.135"/>
-            <geometry>
-                <sphere radius="0.05"/>
-            </geometry>
-        </visual>
-        <collision name='cart_caster_collision_BR'>
-            <origin rpy="0 0 0" xyz="-1.85 -0.35 -0.135"/>
-            <geometry>
-                <sphere radius="0.05"/>
-            </geometry>
-            <surface>
-                <friction>
-                    <ode>
-                        <mu>0</mu>
-                        <mu2>0</mu2>
-                        <slip1>1.0</slip1>
-                        <slip2>1.0</slip2>
-                    </ode>
-                </friction>
-            </surface>
-        </collision>
-        <visual name='cart_caster_visual_BR'>
-            <origin rpy="0 0 0" xyz="-1.85 -0.35 -0.135"/>
-            <geometry>
-                <sphere radius="0.05"/>
-            </geometry>
-        </visual>
+        <xacro:caster name="cart_caster_TL" origin_xyz="-0.95 0.35 -0.135"/>
+        <xacro:caster name="cart_caster_TR" origin_xyz="-0.95 -0.35 -0.135"/>
+        <xacro:caster name="cart_caster_BL" origin_xyz="-1.85 0.35 -0.135"/>
+        <xacro:caster name="cart_caster_BR" origin_xyz="-1.85 -0.35 -0.135"/>
     </link>
     <!-- Cart Wheel -->
-    <link name="left_cart_wheel">
-        <inertial>
-            <mass value="0.2"/>
-            <origin rpy="0 1.5707 1.5707" xyz="0 0 0"/>
-            <inertia ixx="0.000526666666667" ixy="0" ixz="0" iyy="0.000526666666667" iyz="0" izz="0.001"/>
-        </inertial>
-        <collision name="left_cart_wheel_collision">
-            <origin rpy="0 1.5707 1.5707" xyz="0 0 0"/>
-            <geometry>
-                <cylinder length="0.05" radius="0.08"/>
-            </geometry>
-        </collision>
-        <visual name="left_cart_wheel_visual">
-            <origin rpy="0 1.5707 1.5707" xyz="0 0 0"/>
-            <geometry>
-                <cylinder length="0.05" radius="0.08"/>
-            </geometry>
-        </visual>
-    </link>
+    <xacro:link_wheel name="left_cart_wheel" />
     <gazebo reference="left_cart_wheel">
         <mu1>100000.0</mu1>
@@ -394,23 +190,5 @@
         <maxVel>1.0</maxVel>
     </gazebo>
-    <link name="right_cart_wheel">
-        <inertial>
-            <mass value="0.2"/>
-            <origin rpy="0 1.5707 1.5707" xyz="0 0 0"/>
-            <inertia ixx="0.000526666666667" ixy="0" ixz="0" iyy="0.000526666666667" iyz="0" izz="0.001"/>
-        </inertial>
-        <collision name="right_cart_wheel_collision">
-            <origin rpy="0 1.5707 1.5707" xyz="0 0 0"/>
-            <geometry>
-                <cylinder length="0.05" radius="0.08"/>
-            </geometry>
-        </collision>
-        <visual name="right_cart_wheel_visual">
-            <origin rpy="0 1.5707 1.5707" xyz="0 0 0"/>
-            <geometry>
-                <cylinder length="0.05" radius="0.08"/>
-            </geometry>
-        </visual>
-    </link>
+    <xacro:link_wheel name="right_cart_wheel" />
     <gazebo reference="right_cart_wheel">
         <mu1>100000.0</mu1>
@@ -421,20 +199,6 @@
         <maxVel>1.0</maxVel>
     </gazebo>
-    <joint type="continuous" name="joint_left_wheel">
-        <origin rpy="0 0 0" xyz="0 0.38 -0.11"/>
-        <child link="left_wheel"/>
-        <parent link="chassis"/>
-        <axis rpy="0 0 0" xyz="0 1 0"/>
-        <limit effort="10000" velocity="1000"/>
-        <joint_properties damping="1.0" friction="1.0"/>
-    </joint>
-    <joint type="continuous" name="joint_right_wheel">
-        <origin rpy="0 0 0" xyz="0 -0.38 -0.11"/>
-        <child link="right_wheel"/>
-        <parent link="chassis"/>
-        <axis rpy="0 0 0" xyz="0 1 0"/>
-        <limit effort="10000" velocity="1000"/>
-        <joint_properties damping="1.0" friction="1.0"/>
-    </joint>
+    <xacro:joint_wheel name="joint_left_wheel" origin_xyz="0 0.38 -0.11" parent="chassis" child="left_wheel"/>
+    <xacro:joint_wheel name="joint_right_wheel" origin_xyz="0 -0.38 -0.11" parent="chassis" child="right_wheel"/>
     <!-- <joint type="continuous" name="joint_hook">
         <origin rpy="0 0 0" xyz="0 0 0"/>
@@ -459,20 +223,6 @@
         <axis rpy="0 0 0" xyz="0 0 0"/>
     </joint>
-    <joint type="continuous" name="joint_left_cart_wheel">
-        <origin rpy="0 0 0" xyz="-1.4 0.38 -0.11"/>
-        <child link="left_cart_wheel"/>
-        <parent link="cart"/>
-        <axis rpy="0 0 0" xyz="0 1 0"/>
-        <limit effort="10000" velocity="1000"/>
-        <joint_properties damping="1.0" friction="1.0"/>
-    </joint>
-    <joint type="continuous" name="joint_right_cart_wheel">
-        <origin rpy="0 0 0" xyz="-1.4 -0.38 -0.11"/>
-        <child link="right_cart_wheel"/>
-        <parent link="cart"/>
-        <axis rpy="0 0 0" xyz="0 1 0"/>
-        <limit effort="10000" velocity="1000"/>
-        <joint_properties damping="1.0" friction="1.0"/>
-    </joint>
+    <xacro:joint_wheel name="joint_left_cart_wheel" origin_xyz="-1.4 0.38 -0.11" parent="cart" child="left_cart_wheel"/>
+    <xacro:joint_wheel name="joint_right_cart_wheel" origin_xyz="-1.4 -0.38 -0.11" parent="cart" child="right_cart_wheel"/>
     <transmission name="towing_tran">
         <type>transmission_interface/SimpleTransmission</type>

File: amr_dd/models/macros.xacro (robot description, xacro)
@@ -22,3 +22,37 @@
         </link>
     </xacro:macro>
+    <xacro:macro name="joint_wheel" params="name parent child origin_xyz">
+        <joint type="continuous" name="${name}">
+            <origin rpy="0 0 0" xyz="${origin_xyz}"/>
+            <child link="${child}"/>
+            <parent link="${parent}"/>
+            <axis rpy="0 0 0" xyz="0 1 0"/>
+            <limit effort="10000" velocity="1000"/>
+            <joint_properties damping="1.0" friction="1.0"/>
+        </joint>
+    </xacro:macro>
+    <xacro:macro name="caster" params="name origin_xyz">
+        <collision name='${name}_collision'>
+            <origin rpy="0 0 0" xyz="${origin_xyz}"/>
+            <geometry>
+                <sphere radius="0.05"/>}
+            </geometry>
+            <surface>
+                <friction>
+                    <ode>
+                        <mu>0</mu>
+                        <mu2>0</mu2>
+                        <slip1>1.0</slip1>
+                        <slip2>1.0</slip2>
+                    </ode>
+                </friction>
+            </surface>
+        </collision>
+        <visual name='${name}_visual'>
+            <origin rpy="0 0 0" xyz="${origin_xyz}"/>
+            <geometry>
+                <sphere radius="0.05"/>
+            </geometry>
+        </visual>
+    </xacro:macro>
 </robot>

Commit message: laser

File: amr_dd/models/amr_dd.xacro (robot description, xacro)
@@ -199,14 +199,10 @@
         <maxVel>1.0</maxVel>
     </gazebo>
+    <!-- Sensor -->
+    <xacro:laser name="sensor_laser_front"/>
+    <xacro:laser name="sensor_laser_back"/>
+    <!-- Joint -->
     <xacro:joint_wheel name="joint_left_wheel" origin_xyz="0 0.38 -0.11" parent="chassis" child="left_wheel"/>
     <xacro:joint_wheel name="joint_right_wheel" origin_xyz="0 -0.38 -0.11" parent="chassis" child="right_wheel"/>
-    <!-- <joint type="continuous" name="joint_hook">
-        <origin rpy="0 0 0" xyz="0 0 0"/>
-        <child link="hook"/>
-        <parent link="chassis"/>
-        <axis rpy="0 0 0" xyz="0 0 1"/>
-        <limit effort="10000" velocity="1000"/>
-        <joint_properties damping="1.0" friction="1.0"/>
-    </joint> -->
     <joint type="revolute" name="joint_towing">
             <origin rpy="0 0 0" xyz="0 0 0"/>
@@ -231,7 +227,16 @@
         </joint>
         <actuator name="motor_towing">
-            <!-- <hardwareInterface>EffortJointInterface</hardwareInterface> -->
             <mechanicalReduction>1</mechanicalReduction>
         </actuator>
     </transmission>
+    <joint name="joint_sensor_laser_front" type="fixed">
+        <origin xyz="0.45 -0.35 0.165" rpy="0 0 0"/>
+        <parent link="chassis"/>
+        <child link="sensor_laser_front"/>
+    </joint>
+    <joint name="joint_sensor_laser_back" type="fixed">
+        <origin xyz="-0.45 0.35 0.165" rpy="0 0 0"/>
+        <parent link="chassis"/>
+        <child link="sensor_laser_back"/>
+    </joint>
 </robot>

File: amr_dd/models/macros.xacro (robot description, xacro)
@@ -1,4 +1,5 @@
 <?xml version='1.0'?>
 <robot xmlns:xacro="http://www.ros.org/wiki/xacro">
+    <!-- Link Wheel -->
     <xacro:macro name="link_wheel" params="name">
         <link name="${name}">
@@ -22,4 +23,5 @@
         </link>
     </xacro:macro>
+    <!-- Joint Wheel -->
     <xacro:macro name="joint_wheel" params="name parent child origin_xyz">
         <joint type="continuous" name="${name}">
@@ -32,4 +34,5 @@
         </joint>
     </xacro:macro>
+    <!-- Caster -->
     <xacro:macro name="caster" params="name origin_xyz">
         <collision name='${name}_collision'>
@@ -56,3 +59,31 @@
         </visual>
     </xacro:macro>
+    <!-- laser -->
+    <xacro:macro name="laser" params="name">
+        <link name="${name}">
+            <inertial>
+                <mass value="0.05"/>
+                <origin rpy="0 0 0" xyz="0 0 0"/>
+                <xacro:cylinder_inertia mass="0.05" l="0.03" r="0.05" />
+            </inertial>
+            <collision name="${name}_collision">
+                <origin rpy="0 0 0" xyz="0 0 0"/>
+                <geometry>
+                    <cylinder length="0.03" radius="0.05"/>
+                </geometry>
+            </collision>
+            <visual name="${name}_visual">
+                <origin rpy="0 0 0" xyz="0 0 0"/>
+                <geometry>
+                    <cylinder length="0.03" radius="0.05"/>
+                </geometry>
+            </visual>
+        </link>
+    </xacro:macro>
+    <!-- Inertia -->
+    <xacro:macro name="cylinder_inertia" params="mass r l">
+        <inertia  ixx="${mass*(3*r*r+l*l)/12}" ixy = "0" ixz = "0"
+                    iyy="${mass*(3*r*r+l*l)/12}" iyz = "0"
+                    izz="${mass*(r*r)/2}" />
+    </xacro:macro>
 </robot>

Commit message: laser&path

File: amr_dd/models/amr_dd.xacro (robot description, xacro)
@@ -231,10 +231,10 @@
     </transmission>
     <joint name="joint_sensor_laser_front" type="fixed">
-        <origin xyz="0.45 -0.35 0.165" rpy="0 0 0"/>
+        <origin xyz="0.45 0 0.165" rpy="0 0 0"/>
         <parent link="chassis"/>
         <child link="sensor_laser_front"/>
     </joint>
     <joint name="joint_sensor_laser_back" type="fixed">
-        <origin xyz="-0.45 0.35 0.165" rpy="0 0 0"/>
+        <origin xyz="-0.45 0.35 0.165" rpy="0 0 3.14"/>
         <parent link="chassis"/>
         <child link="sensor_laser_back"/>

Commit message: gmapping

File: amr_dd/models/amr_dd.xacro (robot description, xacro)
@@ -4,4 +4,10 @@
     <xacro:include filename="$(find amr_dd)/models/amr_dd.gazebo" />
     <xacro:include filename="$(find amr_dd)/models/macros.xacro" />
+    <link name="base_footprint"/>
+    <joint name="base_joint" type="fixed">
+        <parent link="base_footprint"/>
+        <child link="chassis"/>
+        <origin xyz="0.0 0.0 0.0" rpy="0 0 0"/>
+    </joint>
     <link name='chassis'>
         <!-- pose and inertial -->
@@ -214,9 +220,9 @@
         </joint>
     <joint type="fixed" name="joint_hook">
-        <origin rpy="0 0 0" xyz="0 0 0"/>
-        <child link="cart"/>
-        <parent link="hook"/>
-        <axis rpy="0 0 0" xyz="0 0 0"/>
-    </joint>
+            <origin rpy="0 0 0" xyz="0 0 0"/>
+            <child link="cart"/>
+            <parent link="hook"/>
+            <axis rpy="0 0 0" xyz="0 0 0"/>
+        </joint>
     <xacro:joint_wheel name="joint_left_cart_wheel" origin_xyz="-1.4 0.38 -0.11" parent="cart" child="left_cart_wheel"/>
     <xacro:joint_wheel name="joint_right_cart_wheel" origin_xyz="-1.4 -0.38 -0.11" parent="cart" child="right_cart_wheel"/>
