Commit message: depth camera

File: amr_dd/models/amr_dd.xacro (robot description, xacro)
@@ -4,4 +4,5 @@
     <xacro:include filename="$(find amr_dd)/models/amr_dd.gazebo" />
     <xacro:include filename="$(find amr_dd)/models/macros.xacro" />
+    <xacro:include filename="$(find amr_dd)/urdf/_d435.urdf.xacro" />
     <link name="base_footprint"/>
     <joint name="base_joint" type="fixed">
@@ -208,4 +209,7 @@
     <xacro:laser name="sensor_laser_front"/>
     <xacro:laser name="sensor_laser_back"/>
+    <xacro:sensor_d435 name="camera" topics_ns="camera" parent="chassis" publish_pointcloud="true">
+        <origin xyz="0.51 0 -0.05" rpy="0 -0.2 0" />
+    </xacro:sensor_d435>
     <!-- Joint -->
     <xacro:joint_wheel name="joint_left_wheel" origin_xyz="0 0.38 -0.11" parent="chassis" child="left_wheel"/>
@@ -230,5 +234,5 @@
         <type>transmission_interface/SimpleTransmission</type>
         <joint type="revolute" name="joint_towing">
-            <hardwareInterface>EffortJointInterface</hardwareInterface>
+            <hardwareInterface>hardware_interface/EffortJointInterface</hardwareInterface>
         </joint>
         <actuator name="motor_towing">
